File: PCB/adc.kicad_sch (KiCad schematic)
At the start: 0 parts

Commit message: updated schematics
Parts:
- added C35: 1uF, symbol Device:C_Small
- added C36, C37, C39: 10uF, symbol Device:C_Polarized_Small
- added C38: 1uF, symbol Device:C_Polarized_Small
- added CN1: PJ-358H-B, easyeda2kicad:AUDIO-TH_PJ-358H-B, symbol easyeda2kicad:PJ-358H-B
- added U18: PCM1809IRTER, easyeda2kicad:WQFN-20_L3.0-W3.0-P0.50-TL-EP1.4, symbol easyeda2kicad:PCM1809IRTER
Connections:
- new net: C37.1, U18.14 (DREG)
- new net: C36.1, U18.17 (AREG)
- new net: C35.1, U18.18 (VREF)
- new net AVDD_3V3: C38.1, U18.16 (AVDD)
- new net BCKO: U18.7 (BCLK)
- new net DOUT: U18.6 (SDOUT)
- new net GND: C35.2, C36.2, C37.2, C38.2, C39.2, CN1.3 (TSW), U18.10 (VSS), U18.11 (MD1), U18.12 (MD0), U18.13 (MSZ), U18.15 (VSS), U18.19 (FMT0), U18.2 (IN1M), U18.20 (VSS), U18.21 (EP), U18.4 (IN2M), U18.5 (VSS)
- new net IOVDD_3V3: C39.1, U18.9 (IOVDD)
- new net LRCKO: U18.8 (FSYNC)
- new net Left Audio: CN1.2 (Tip), U18.1 (IN1P)
- new net Right Audio: CN1.5 (Ring), U18.3 (IN2P)
- new net Sleeve: CN1.1 (Sleeve)
- new net Tip Switch IN: CN1.4 (TSW)
