File: PCB/raspi.kicad_sch (KiCad schematic)
At the start: 5 parts, among them Q1 AO3400A, U12 RASPBERRY_PI_ZERO_2_W

Commit message: updated schematics
Parts:
- U12: footprint RASPBERRY_PI_ZERO_2_W:RASPBERRY_PI_ZERO_2_W -> RASPBERRY_PI_ZERO_2_W:MODULE_RASPBERRY_PI_ZERO_2_W
Changed lines of the file:
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@@
 			)
 		)
-		(property "Footprint" "RASPBERRY_PI_ZERO_2_W:RASPBERRY_PI_ZERO_2_W"
+		(property "Footprint" "RASPBERRY_PI_ZERO_2_W:MODULE_RASPBERRY_PI_ZERO_2_W"
 			(at 148.59 91.44 0)
 			(effects
