File: PCB/esp32.kicad_sch (KiCad schematic)
At the start: 29 parts, among them J1 UART, SW1 Boot, SW2 Reset, U4 ESP32-S3-WROOM-1, U8 GT-USB-7010ASV, U9 SGM2212-3.3XKC3G

Commit message: Initial commit of project source code
Other:
- moved on the sheet: C10, C11, C7, C8, C9, D8, D9, U9

Commit message: updated schematics
Parts:
- removed C10, C4, C8, C9: 10uF, symbol Device:C_Small
- removed C11, C7: 0.1uF, symbol Device:C_Small
- removed D1, D9: LESD5D5.0CT1G, Diode_SMD:D_SOD-523, symbol Device:D_TVS
- removed D4, D8: 1N5819HW-7-F, Diode_SMD:D_SOD-123, symbol Diode:1N5819
- removed U9: SGM2212-3.3XKC3G, easyeda2kicad:SOT-223-3_L6.5-W3.4-P2.30-LS7.0-BR, symbol easyeda2kicad:SGM2212-3.3XKC3G_TR_C3294699
- U4: footprint RF_Module:ESP32-S3-WROOM-1U -> RF_Module:ESP32-S3-WROOM-1
Connections:
- net +3V3 renamed DVDD_3V3
- net DVDD_3V3: now also R2.1
- net ESP_3V3: no longer names the net of R1.2, U4.2 (3V3)
- net ESP_3V3: no longer R2.1
- net VBUSB: no longer names the net of U8.A4 (VBUS)
- net VCC_5V renamed +5V
- net VIN 5V: no longer names the net of U8.B4 (VBUS)
- no-connect marks 2 -> 4

Commit message: Saving my work on PCB and other files
Parts:
- C2: value 0.1uF -> 10uF
- U4: value ESP32-S3-WROOM-1 -> ESP32-S3-WROOM-1U-N8
Changed lines of the file:
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@@
 			)
 		)
-		(property "Value" "0.1uF"
+		(property "Value" "10uF"
 			(at 140.208 56.388 0)
 			(effects
@@
 			)
 		)
-		(property "Value" "ESP32-S3-WROOM-1"
+		(property "Value" "ESP32-S3-WROOM-1U-N8"
 			(at 155.956 70.612 0)
 			(effects
