File: HID/esp32_hid.kicad_sch (KiCad schematic)
At the start: 25 parts, among them J1 UART, J2 PWR, J3 DATA, J4 <- Encoder, J5 Display, SW1 Boot, SW2 Reset, U1 AMS1117-3.3, U2 ESP32-S3-WROOM-1U-N16R8

Commit message: Update PCB/Schematic files, scripts and just refractured
Parts:
- removed J1: UART, Connector_PinHeader_2.54mm:PinHeader_1x04_P2.54mm_Vertical, symbol Connector_Generic:Conn_01x04
- added J1: UART, Connector_PinHeader_2.54mm:PinHeader_1x05_P2.54mm_Vertical, symbol Connector_Generic:Conn_01x05
- added J6: UART 2, Connector_PinHeader_2.54mm:PinHeader_1x03_P2.54mm_Vertical, symbol Connector_Generic:Conn_01x03
- added Q1, Q2: L8050QLT1G, Package_TO_SOT_SMD:SOT-23, symbol Transistor_BJT:Q_NPN_BEC
- added R10, R11: 82R, Resistor_SMD:R_0603_1608Metric, symbol Device:R
- added R12, R8, R9: 0R, Resistor_SMD:R_0603_1608Metric, symbol Device:R
- added R13, R14, R15, R16, R6, R7: 10k, Resistor_SMD:R_0603_1608Metric, symbol Device:R
- renumbered C10 to C11
Connections:
- net 3VV3: now also J1.2 (Pin_2), R13.2, R14.2, R15.2, R16.2
- net 5V: now also J4.2 (Pin_2), J4.3 (Pin_3), J6.2 (Pin_2); no longer J4.1 (Pin_1)
- net CHIP_PU: now also R9.2
- net CTP_INT: now also R16.1
- net CTP_RST: now also R15.1
- net ESP_CS: now also J3.4 (Pin_4); no longer J3.3 (Pin_3)
- net ESP_MISO: now also J3.3 (Pin_3); no longer J3.4 (Pin_4)
- net GND: now also J4.1 (Pin_1), J1.1 (Pin_1), J6.1 (Pin_1); no longer J4.10 (Pin_10), J4.2 (Pin_2)
- net GPIO0: now also R8.2
- net INT: now also J4.10 (Pin_10); no longer J4.9 (Pin_9)
- net LCD_CS: now also R13.1
- net LCD_RST: now also R14.1
- net LED_DATA: now also J4.5 (Pin_5); no longer J4.3 (Pin_3)
- net MISO: now also R12.1; no longer U2.19 (IO11)
- net MOSI: now also R10.1; no longer U2.20 (IO12)
- net SCK: now also R11.1; no longer U2.21 (IO13)
- net SCL: now also J4.7 (Pin_7); no longer J4.5 (Pin_5)
- net SDA: now also J4.9 (Pin_9); no longer J4.7 (Pin_7)
- net U0RXD: now also J1.3 (Pin_3)
- net U0TXD: now also J1.4 (Pin_4)
- new net: Q1.1 (B), R6.2
- new net: Q1.3 (C), R9.1
- new net: R12.2, U2.21 (IO13)
- new net: Q2.1 (B), R7.2
- new net: R11.2, U2.20 (IO12)
- new net: Q2.3 (C), R8.1
- new net: R10.2, U2.19 (IO11)
- new net DTR: J1.5 (Pin_5), Q2.2 (E), R6.1
- new net RTS: J6.3 (Pin_3), Q1.2 (E), R7.1
Other:
- note added: "Auto program"
- moved on the sheet: C1, R1
